File: Eagle/Projects/Monoblink_Main/Monoblink_attiny85/Monoblink.sch (EAGLE design)
At the start: 6 parts, among them U1 ATTINY85

Commit message: monoblink main
Parts:
- removed J1: (no value), Monoblink:BATT_CONN
- added C2: 100n, Monoblink:C-USC0603
- added GND, PB0, PB1, PB2, PB3, PB4, PB5, VCC: TESTPAD_PROG_BOARD, Monoblink:TESTPAD_PROG_BOARD
- added R1: 50, Monoblink:R-US_R0603
- added R2: 200, Monoblink:R-US_R0603
- added R3: 100, Monoblink:R-US_R0603
- added R4: 10K, Monoblink:R-US_R0603
- added R5, R6: 100K, Monoblink:R-US_R0603
- added U$3: BATT_TH, Monoblink:BATT_TH
- added U$4: SNSR_CONN, Monoblink:SNSR_CONN
- C1: value (none) -> 100n; device Monoblink:C-USC0805 -> Monoblink:C-USC0603
Connections:
- removed net LED_DATA_IN: LED1.DIN, U1.PB2
- new net PB0: LED1.DIN, PB0.1, U1.PB0
- new net PB1: PB1.1, R6.1, U1.PB1
- new net PB2: PB2.1, R5.2, U1.PB2
- new net PB3: PB3.1, R2.1, U1.PB3
- new net PB4: PB4.1, R3.1, U1.PB4
- new net PB5: PB5.1, R1.1, U1.PB5
- new net SENSOR_OUT: C2.1, R4.1, R5.1, U$4.SNSR
- net GND: now also C2.2, GND.1, U$3.GND, U$4.GND; no longer J1.-
- net PIEZO_IN: now also R1.2, R2.2, R3.2; no longer U1.PB0
- net RF_DATA_OUT: now also R6.2; no longer U1.PB1
- net VCC: now also R4.2, U$3.VBAT, VCC.1; no longer J1.+
Other:
- note added: "Il faut ajouter des résistances sur RF_DATA_OUT et SENSOR_OUT pour que le programmeur puisse imposer les niveaux"
- moved on the sheet: U1
