File: Eagle/Projects/Monoblink_Main/Monoblink_Wifi_V2.2/monoblink_wifi_v2.sch (EAGLE design)
At the start: 25 parts

Commit message: dio commander
Parts:
- CLK, DAT, GND, VCC: value TESTPAD_PROG -> TESTPAD_PROGSPRING_PIN; device monoblink_wifi:TESTPAD_PROG -> monoblink_wifi:TESTPAD_PROGSPRING_PIN
