File: Eagle/Projects/Electrode_Tester_v1.0/electrode_tester.brd (EAGLE design)
At the start: 63.5 x 34.3 mm, 56 parts, among them U1 ADS1248, U2 LMP7702MM/NOPBVSSOP

Commit message: git update
Other:
- board size 63.5 x 34.3 mm -> 47 x 22.9 mm
